File: KAPTON HEATER.kicad_pcb (KiCad board)
At the start: 2 copper layers, 20 parts, among them J1 Conn_01x02_Pin, J5 10090926-P154XLF

Commit message: fixing repo
Parts:
- R1: footprint Resistor_THT:R_Axial_DIN0204_L3.6mm_D1.6mm_P2.54mm_Vertical -> Resistor_SMD:R_0201_0603Metric; moved to B.Cu
- R2, R3, R4, R5, R6, R7, R8, R9: footprint Resistor_SMD:R_0805_2012Metric -> Resistor_SMD:R_0201_0603Metric; moved to B.Cu
- TH1, TH2, TH3, TH4, TH5, TH6, TH7, TH8, TH9: footprint Resistor_SMD:R_0402_1005Metric_Pad0.72x0.64mm_HandSolder -> Resistor_THT:R_Array_SIP4
- moved TH9 599.7 mm to (376.5, 195.1), turned to 90 degrees
- moved TH8 565.9 mm to (520.5, 193.5), turned to 90 degrees
- moved TH7 562.3 mm to (637.5, 194.1), turned to 90 degrees
- moved TH4 444.9 mm to (386.0, 349.4), turned to 90 degrees
- moved TH5 405.9 mm to (520.5, 348.9), turned to 90 degrees
- moved TH6 405.9 mm to (637.5, 349.5), turned to 90 degrees
- moved TH1 266.4 mm to (385.5, 564.1), turned to 90 degrees
- moved TH2 190.1 mm to (520.5, 564.7), turned to 90 degrees
- moved TH3 189.0 mm to (637.5, 564.6), turned to 90 degrees
- moved R1 134.0 mm to (566.0, 618.3), turned to 90 degrees
- moved R9 121.7 mm to (591.3, 618.3), turned to 90 degrees
- moved R8 119.3 mm to (588.2, 618.3), turned to 90 degrees
- moved R7 117.1 mm to (585.0, 618.3), turned to 90 degrees
- moved R6 114.9 mm to (581.8, 618.3), turned to 90 degrees
- moved R5 112.9 mm to (578.5, 618.3), turned to 90 degrees
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Connections:
- J1 pad 2: 24V -> Return
- R1 pad 1: Net-(R1-Pad1) -> TH5
- TH5 pad 2: Net-(R1-Pad1) -> TH5
Routing:
- net 5V: track 0.00 -> 1264.1 mm, vias 0 -> 2
- net TH9: track 0.00 -> 674.1 mm, vias 0 -> 9
- net TH7: track 0.00 -> 511.0 mm, vias 0 -> 3
- net TH8: track 0.00 -> 496.3 mm, vias 0 -> 9
- net TH4: track 0.00 -> 478.1 mm, vias 0 -> 3
- net TH6: track 0.00 -> 357.7 mm, vias 0 -> 3
- net TH5: track 0.00 -> 339.4 mm, vias 0 -> 4
- net TH1: track 0.00 -> 270.3 mm, vias 0 -> 4
- net TH2: track 0.00 -> 128.0 mm, vias 0 -> 2
- net TH3: track 0.00 -> 126.1 mm, vias 0 -> 4
- net GND: track 0.00 -> 86.7 mm, vias 0 -> 3
- net 24V: track 15519.6 -> 15560.5 mm
- net Net-(U1-SOURCE): track 4.38 -> 0.00 mm
- net (no net): track 2.34 -> 0.00 mm
Other:
- board outline added: 322 x 544 mm
