File: KAPTON HEATER.kicad_sch (KiCad schematic)
At the start: 21 parts, among them J1 Conn_01x02_Pin, J5 10090926-P154XLF

Commit message: fixing repo
Connections:
- net TH5: now also R1.1, TH5.2
Changed lines of the file:
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@@
 	(global_label "TH5"
 		(shape input)
-		(at 185.42 100.33 180)
+		(at 186.69 100.33 180)
 		(fields_autoplaced yes)
 		(effects
@@
 		)
 		(property "Intersheetrefs" "${INTERSHEET_REFS}"
-			(at 178.9272 100.33 0)
+			(at 180.1972 100.33 0)
 			(effects
 				(font
